File: Solar Charger 2020 PCB/SolarCharger2020.sch (KiCad schematic (older format))
At the start: 16 parts, among them P1 LiPo OUTPUT, P3 PV INPUT, U1 BQ24210

Commit message: Updated instructions
Other:
- note added: "Ts pulled high for solar charging applications\nLimited current mode to ensure battery temperature OK\nPull high with 100k \n\nVDPM\nKept open for load tracking, such as solar PV \nVDPM to ground using\nRVDPM= (VBUS_DPM–VBUS_DPM_1)/KVBUS_DPM \n= (4.6 V - 3.5 V) / ( 0.15V/kΩ) = 7.333kΩ → 7.32kΩ \nclosest 1% resistor\n\nIset\n2W of solar PV gives 400mA maximum\nRiset = Kiset/Iout Iout = 400mA. Kise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"
- note removed: "DC/DC Converter for 5V output\nWant it to switch on when current drawn?\nIs this possible?\nUsing: MIC2288YD5-TR"
- note removed: "Recharge LiPo fro USB if available\n"
- note removed: "Ts pulled high for solar charing applications\nLimited current mode to ensure battery temperature OK\nPull high with 100k \n\nVDPM\nKept open for load tracking, such as solar PV \nVDPM to ground using\nRVDPM= (VBUS_DPM–VBUS_DPM_1)/KVBUS_DPM \n= (4.6 V - 3.5 V) / ( 0.15V/kΩ) = 7.333kΩ → 7.32kΩ \nclosest 1% resistor\n\nIset\n2W of solar PV gives 400mA maximum\nRiset = Kiset/Iout Iout = 400mA. Kiset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"
Changed lines of the file:
@@
 EESchema Schematic File Version 4
-LIBS:power
-LIBS:device
-LIBS:transistors
-LIBS:conn
-LIBS:regul
-LIBS:74xx
-LIBS:cmos4000
-LIBS:adc-dac
-LIBS:memory
-LIBS:xilinx
-LIBS:microcontrollers
-LIBS:dsp
-LIBS:microchip
-LIBS:analog_switches
-LIBS:motorola
-LIBS:texas
-LIBS:intel
-LIBS:audio
-LIBS:interface
-LIBS:digital-audio
-LIBS:philips
-LIBS:display
-LIBS:cypress
-LIBS:siliconi
-LIBS:opto
-LIBS:atmel
-LIBS:contrib
-LIBS:valves
-LIBS:matts_components
 LIBS:SolarCharger2020-cache
 EELAYER 29 0
@@
 	1    0    0    -1
 $EndComp
-Text Notes 3150 4800 0    60   ~ 0
-Ts pulled high for solar charing applications\nLimited current mode to ensure battery temperature OK\nPull high with 100k \n\nVDPM\nKept open for load tracking, such as solar PV \nVDPM to ground using\nRVDPM= (VBUS_DPM–VBUS_DPM_1)/KVBUS_DPM \n= (4.6 V - 3.5 V) / ( 0.15V/kΩ) = 7.333kΩ → 7.32kΩ \nclosest 1% resistor\n\nIset\n2W of solar PV gives 400mA maximum\nRiset = Kiset/Iout Iout = 400mA. Kiset = 395Aohm. Riset = 987.5. \nClose to 1k\n\nEN tied to PG as load mode never used
+Text Notes 2950 6550 0    60   ~ 0
+Ts pulled high for solar charging applications\nLimited current mode to ensure battery temperature OK\nPull high with 100k \n\nVDPM\nKept open for load tracking, such as solar PV \nVDPM to ground using\nRVDPM= (VBUS_DPM–VBUS_DPM_1)/KVBUS_DPM \n= (4.6 V - 3.5 V) / ( 0.15V/kΩ) = 7.333kΩ → 7.32kΩ \nclosest 1% resistor\n\nIset\n2W of solar PV gives 400mA maximum\nRiset = Kiset/Iout Iout = 400mA. Kiset = 395Aohm. Riset = 987.5. \nClose to 1k\n\nEN tied to PG as load mode never used
 Wire Wire Line
 	3400 2150 3250 2150
@@
 Wire Wire Line
 	1700 1550 2050 1550
-Text Notes 7600 4800 0    60   ~ 0
-DC/DC Converter for 5V output\nWant it to switch on when current drawn?\nIs this possible?\nUsing: MIC2288YD5-TR
-Text Notes 7550 3650 0    60   ~ 0
-Recharge LiPo fro USB if available\n
 Wire Wire Line
 	4850 1550 5150 1550
